File: PCB/PCB.kicad_pcb (KiCad board)
At the start: 2 copper layers, 41 x 42.5 mm, 30 parts, among them J1 Conn_01x02_Socket, J2 Conn_01x04_Socket, Q1 NMOS, Q2 NMOS, Q3 NMOS, Q4 NMOS, Q5 NMOS, Q6 NMOS, U1 Teensy4.0, U2 L7805

Commit message: Stupid dumb fix
Also did geographical reannotation
Parts:
- renumbered C3 to C1, C1 to C3, Q6 to Q1, Q5 to Q2, Q4 to Q3, Q2 to Q4, Q3 to Q5, Q1 to Q6, R10 to R1, R6 to R10, R9 to R11, R7 to R12, R8 to R13, R5 to R14, R4 to R15, R15 to R2, R1 to R3, R3 to R4, R13 to R5, R14 to R6, R2 to R7, R12 to R8, R11 to R9
Routing:
- net PDM Clock: track 22.6 -> 24.4 mm
Changed lines of the file:
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@@
 			(pinfunction "GND")
 			(pintype "power_in")
-			(zone_connect 0)
 			(options
 				(clearance outline)
@@
 		(descr "Resistor SMD 0603 (1608 Metric), square (rectangular) end terminal, IPC-7351 nominal, (Body size source: IPC-SM-782 page 72, https://www.pcb-3d.com/wordpress/wp-content/uploads/ipc-sm-782a_amendment_1_and_2.pdf), generated with kicad-footprint-generator")
 		(tags "resistor")
-		(property "Reference" "R10"
+		(property "Reference" "R1"
 			(at 0 1.5 0)
 			(layer "B.SilkS")
@@
 		(descr "SC-59, https://lib.chipdip.ru/images/import_diod/original/SOT-23_SC-59.jpg")
 		(tags "SC-59")
-		(property "Reference" "Q1"
+		(property "Reference" "Q6"
 			(at 2.2 1.5 0)
 			(layer "B.SilkS")
@@
 		(descr "Resistor SMD 0603 (1608 Metric), square (rectangular) end terminal, IPC-7351 nominal, (Body size source: IPC-SM-782 page 72, https://www.pcb-3d.com/wordpress/wp-content/uploads/ipc-sm-782a_amendment_1_and_2.pdf), generated with kicad-footprint-generator")
 		(tags "resistor")
-		(property "Reference" "R6"
+		(property "Reference" "R10"
 			(at 0 1.43 0)
 			(layer "B.SilkS")
@@
 		(descr "Resistor SMD 0603 (1608 Metric), square (rectangular) end terminal, IPC-7351 nominal, (Body size source: IPC-SM-782 page 72, https://www.pcb-3d.com/wordpress/wp-content/uploads/ipc-sm-782a_amendment_1_and_2.pdf), generated with kicad-footprint-generator")
 		(tags "resistor")
-		(property "Reference" "R15"
+		(property "Reference" "R2"
 			(at -0.175 -1.5 0)
 			(layer "B.SilkS")
@@
 		(descr "Capacitor SMD 0603 (1608 Metric), square (rectangular) end terminal, IPC-7351 nominal, (Body size source: IPC-SM-782 page 76, https://www.pcb-3d.com/wordpress/wp-content/uploads/ipc-sm-782a_amendment_1_and_2.pdf), generated with kicad-footprint-generator")
 		(tags "capacitor")
-		(property "Reference" "C1"
+		(property "Reference" "C3"
 			(at -2.725 0 90)
 			(layer "B.SilkS")
@@
 		(descr "Resistor SMD 0603 (1608 Metric), square (rectangular) end terminal, IPC-7351 nominal, (Body size source: IPC-SM-782 page 72, https://www.pcb-3d.com/wordpress/wp-content/uploads/ipc-sm-782a_amendment_1_and_2.pdf), generated with kicad-footprint-generator")
 		(tags "resistor")
-		(property "Reference" "R9"
+		(property "Reference" "R11"
 			(at 0 1.43 90)
 			(layer "B.SilkS")
@@
 		(descr "Resistor SMD 0603 (1608 Metric), square (rectangular) end terminal, IPC-7351 nominal, (Body size source: IPC-SM-782 page 72, https://www.pcb-3d.com/wordpress/wp-content/uploads/ipc-sm-782a_amendment_1_and_2.pdf), generated with kicad-footprint-generator")
 		(tags "resistor")
-		(property "Reference" "R7"
+		(property "Reference" "R12"
 			(at 0 1.43 90)
 			(layer "B.SilkS")
@@
 		(descr "SC-59, https://lib.chipdip.ru/images/import_diod/original/SOT-23_SC-59.jpg")
 		(tags "SC-59")
-		(property "Reference" "Q2"
+		(property "Reference" "Q4"
 			(at 2.2 2 0)
 			(layer "B.SilkS")
@@
 		(descr "Resistor SMD 0603 (1608 Metric), square (rectangular) end terminal, IPC-7351 nominal, (Body size source: IPC-SM-782 page 72, https://www.pcb-3d.com/wordpress/wp-content/uploads/ipc-sm-782a_amendment_1_and_2.pdf), generated with kicad-footprint-generator")
 		(tags "resistor")
-		(property "Reference" "R5"
+		(property "Reference" "R14"
 			(at 0 1.43 90)
 			(layer "B.SilkS")
@@
 		(descr "Resistor SMD 0603 (1608 Metric), square (rectangular) end terminal, IPC-7351 nominal, (Body size source: IPC-SM-782 page 72, https://www.pcb-3d.com/wordpress/wp-content/uploads/ipc-sm-782a_amendment_1_and_2.pdf), generated with kicad-footprint-generator")
 		(tags "resistor")
-		(property "Reference" "R1"
+		(property "Reference" "R3"
 			(at 0 1.43 90)
 			(layer "B.SilkS")
@@
 		(descr "Resistor SMD 0603 (1608 Metric), square (rectangular) end terminal, IPC-7351 nominal, (Body size source: IPC-SM-782 page 72, https://www.pcb-3d.com/wordpress/wp-content/uploads/ipc-sm-782a_amendment_1_and_2.pdf), generated with kicad-footprint-generator")
 		(tags "resistor")
-		(property "Reference" "R3"
+		(property "Reference" "R4"
 			(at 2.5 0.35 180)
 			(layer "B.SilkS")
@@
 		(descr "Resistor SMD 0603 (1608 Metric), square (rectangular) end terminal, IPC-7351 nominal, (Body size source: IPC-SM-782 page 72, https://www.pcb-3d.com/wordpress/wp-content/uploads/ipc-sm-782a_amendment_1_and_2.pdf), generated with kicad-footprint-generator")
 		(tags "resistor")
-		(property "Reference" "R13"
+		(property "Reference" "R5"
 			(at -0.135 -1.5 0)
 			(layer "B.SilkS")
@@
 		(descr "Resistor SMD 0603 (1608 Metric), square (rectangular) end terminal, IPC-7351 nominal, (Body size source: IPC-SM-782 page 72, https://www.pcb-3d.com/wordpress/wp-content/uploads/ipc-sm-782a_amendment_1_and_2.pdf), generated with kicad-footprint-generator")
 		(tags "resistor")
-		(property "Reference" "R4"
+		(property "Reference" "R15"
 			(at 0 1.43 0)
 			(layer "B.SilkS")
@@
 		(descr "Resistor SMD 0603 (1608 Metric), square (rectangular) end terminal, IPC-7351 nominal, (Body size source: IPC-SM-782 page 72, https://www.pcb-3d.com/wordpress/wp-content/uploads/ipc-sm-782a_amendment_1_and_2.pdf), generated with kicad-footprint-generator")
 		(tags "resistor")
-		(property "Reference" "R14"
+		(property "Reference" "R6"
 			(at 0 1.43 0)
 			(layer "B.SilkS")
@@
 		(descr "SC-59, https://lib.chipdip.ru/images/import_diod/original/SOT-23_SC-59.jpg")
 		(tags "SC-59")
-		(property "Reference" "Q6"
+		(property "Reference" "Q1"
 			(at 0.35 -2.5 0)
 			(layer "B.SilkS")
@@
 		(descr "Resistor SMD 0603 (1608 Metric), square (rectangular) end terminal, IPC-7351 nominal, (Body size source: IPC-SM-782 page 72, https://www.pcb-3d.com/wordpress/wp-content/uploads/ipc-sm-782a_amendment_1_and_2.pdf), generated with kicad-footprint-generator")
 		(tags "resistor")
-		(property "Reference" "R8"
+		(property "Reference" "R13"
 			(at 0 1.43 0)
 			(layer "B.SilkS")
@@
 		(descr "Resistor SMD 0603 (1608 Metric), square (rectangular) end terminal, IPC-7351 nominal, (Body size source: IPC-SM-782 page 72, https://www.pcb-3d.com/wordpress/wp-content/uploads/ipc-sm-782a_amendment_1_and_2.pdf), generated with kicad-footprint-generator")
 		(tags "resistor")
-		(property "Reference" "R2"
+		(property "Reference" "R7"
 			(at -2.5 -0.85 180)
 			(layer "B.SilkS")
@@
 		(descr "SC-59, https://lib.chipdip.ru/images/import_diod/original/SOT-23_SC-59.jpg")
 		(tags "SC-59")
-		(property "Reference" "Q5"
+		(property "Reference" "Q2"
 			(at 0 -2.5 0)
 			(layer "B.SilkS")
@@
 		(descr "Resistor SMD 0603 (1608 Metric), square (rectangular) end terminal, IPC-7351 nominal, (Body size source: IPC-SM-782 page 72, https://www.pcb-3d.com/wordpress/wp-content/uploads/ipc-sm-782a_amendment_1_and_2.pdf), generated with kicad-footprint-generator")
 		(tags "resistor")
-		(property "Reference" "R12"
+		(property "Reference" "R8"
 			(at 0 1.43 0)
 			(layer "B.SilkS")
@@
 		(descr "Resistor SMD 0603 (1608 Metric), square (rectangular) end terminal, IPC-7351 nominal, (Body size source: IPC-SM-782 page 72, https://www.pcb-3d.com/wordpress/wp-content/uploads/ipc-sm-782a_amendment_1_and_2.pdf), generated with kicad-footprint-generator")
 		(tags "resistor")
-		(property "Reference" "R11"
+		(property "Reference" "R9"
 			(at -0.175 -1.5 0)
 			(layer "B.SilkS")
@@
 		(descr "SC-59, https://lib.chipdip.ru/images/import_diod/original/SOT-23_SC-59.jpg")
 		(tags "SC-59")
-		(property "Reference" "Q4"
+		(property "Reference" "Q3"
 			(at 1 -2.5 0)
 			(layer "B.SilkS")
@@
 		(descr "SC-59, https://lib.chipdip.ru/images/import_diod/original/SOT-23_SC-59.jpg")
 		(tags "SC-59")
-		(property "Reference" "Q3"
+		(property "Reference" "Q5"
 			(at 1.7 2.5 0)
 			(layer "B.SilkS")
@@
 		(descr "Capacitor SMD 0603 (1608 Metric), square (rectangular) end terminal, IPC-7351 nominal, (Body size source: IPC-SM-782 page 76, https://www.pcb-3d.com/wordpress/wp-content/uploads/ipc-sm-782a_amendment_1_and_2.pdf), generated with kicad-footprint-generator")
 		(tags "capacitor")
-		(property "Reference" "C3"
+		(property "Reference" "C1"
 			(at 0 1.43 0)
 			(layer "B.SilkS")
@@
 	)
 	(segment
-		(start 171.5 54)
-		(end 166.5 59)
+		(start 167.5 59)
+		(end 169.5 57)
+		(width 0.2)
+		(layer "F.Cu")
+		(net 10)
+	)
+	(segment
+		(start 161 59)
+		(end 167.5 59)
+		(width 0.2)
+		(layer "F.Cu")
+		(net 10)
+	)
+	(segment
+		(start 169.5 55)
+		(end 171 53.5)
 		(width 0.2)
 		(layer "F.Cu")
@@
 	)
 	(segment
-		(start 166.5 59)
-		(end 161 59)
+		(start 174.58 53.995)
+		(end 174.58 54.96)
 		(width 0.2)
 		(layer "F.Cu")
@@
 	)
 	(segment
-		(start 174.17 54)
-		(end 171.5 54)
+		(start 169.5 57)
+		(end 169.5 55)
 		(width 0.2)
 		(layer "F.Cu")
@@
 	)
 	(segment
-		(start 174.58 54.41)
-		(end 174.17 54)
+		(start 174.085 53.5)
+		(end 174.58 53.995)
 		(width 0.2)
 		(layer "F.Cu")
@@
 	)
 	(segment
-		(start 174.58 54.96)
-		(end 174.58 54.41)
+		(start 171 53.5)
+		(end 174.085 53.5)
 		(width 0.2)
 		(layer "F.Cu")

Commit message: discussed changes
Parts:
- added R7: 84.5, Resistor_SMD:R_0603_1608Metric, B.Cu at (176.5, 56.0)
- moved R11 0.51 mm to (172.9, 67.0)
- renumbered Q5 to Q4, Q4 to Q5, R8 to R1, R7 to R10, R13 to R11, R10 to R12, R15 to R13, R11 to R14, R12 to R15, R14 to R16, R6 to R3, R1 to R4, R9 to R5, R5 to R6, R3 to R8, R4 to R9
Connections:
- MK1 pad 1: PDM Data -> Net-(MK1-DATA)
- MK1 pad 4: +3.3V -> GND
Routing:
- net Net-(MK1-DATA): track 0.00 -> 2.54 mm, vias 0 -> 1
- net +3.3V: track 32.0 -> 30.3 mm
- net PDM Data: track 36.7 -> 35.7 mm, vias 0 -> 1
- net PDM Clock: track 24.4 -> 25.2 mm
- net Net-(Q4-G): track 5.48 -> 4.97 mm
Other:
- board text added: "Flux"
- board text added: "R1.0"
