File: PCB/PCB.kicad_sch (KiCad schematic)
At the start: 0 parts

Commit message: schematic complete
Parts:
- added C1: 0.33 uF, symbol Device:C
- added C2: 0.1 uF, symbol Device:C
- added D1: LED_RGBA, symbol Device:LED_RGBA
- added J1: Conn_01x02_Socket, symbol Connector:Conn_01x02_Socket
- added J2: Conn_01x04_Socket, symbol Connector:Conn_01x04_Socket
- added MK1: IM69D130, Sensor_Audio:Infineon_PG-LLGA-5-1, symbol Sensor_Audio:IM69D130
- added Q1, Q2, Q3, Q4, Q5, Q6: NMOS, symbol Simulation_SPICE:NMOS
- added R1: 150, symbol Device:R
- added R10, R11, R12, R4, R6, R8: 1K, symbol Device:R
- added R13, R14, R15, R5, R7, R9: 10K, symbol Device:R
- added R2, R3: 84.5, symbol Device:R
- added U1: Teensy4.0, Custom:Teensy40, symbol Custom:Teensy4.0
- added U2: L7805, symbol Regulator_Linear:L7805
Connections:
- new net: Q4.1 (D), R1.1
- new net: D1.1 (RK), R1.2
- new net: Q6.2 (G), R12.2, R15.2
- new net: Q2.2 (G), R6.2, R7.2
- new net: Q5.2 (G), R11.2, R14.2
- new net: Q4.2 (G), R10.2, R13.2
- new net: Q6.1 (D), R3.1
- new net: D1.3 (BK), R3.2
- new net: Q1.2 (G), R4.2, R5.2
- new net: D1.2 (GK), R2.2
- new net: Q3.2 (G), R8.2, R9.2
- new net: Q5.1 (D), R2.1
- new net +12V: C1.1, J1.1 (Pin_1), J2.1 (Pin_1), U2.1 (IN)
- new net +3.3V: MK1.2 (VDD), U1.31 (3V3)
- new net +5V: C2.2, D1.4 (A), U1.33 (VIN), U2.3 (OUT)
- new net Blue Power: J2.4 (Pin_4), Q3.1 (D)
- new net Blue Signal: R12.1, R8.1, U1.20 (13_SCK_CRX1_LED)
- new net GND: C1.2, C2.1, J1.2 (Pin_2), MK1.5 (GND), Q1.3 (S), Q2.3 (S), Q3.3 (S), Q4.3 (S), Q5.3 (S), Q6.3 (S), R13.1, R14.1, R15.1, R5.1, R7.1, R9.1, U1.1 (GND), U1.32 (GND), U2.2 (GND)
- new net Green Power: J2.3 (Pin_3), Q2.1 (D)
- new net Green Signal: R11.1, R6.1, U1.21 (14_A0_TX3_SPDIF_OUT)
- new net PDM Clock: MK1.3 (CLOCK), U1.28 (21_A7_RX5_BCLK1)
- new net PDM Data: MK1.1 (DATA), U1.10 (8_TX2_IN1)
- new net Red Power: J2.2 (Pin_2), Q1.1 (D)
- new net Red Signal: R10.1, R4.1, U1.22 (15_A1_RX3_SPDIF_IN)
- no-connect marks 0 -> 20

Commit message: everything done except stupid 1 issue
Parts:
- added C3: 0.1 uF, Capacitor_SMD:C_0603_1608Metric, symbol Device:C
- C1, C2: footprint (none) -> Capacitor_SMD:C_0603_1608Metric
- D1: footprint (none) -> Custom:150066M153000
- J1: footprint (none) -> Custom:2.1x5.5_Barrel_Jack
- J2: footprint (none) -> TerminalBlock_Phoenix:TerminalBlock_Phoenix_MKDS-1,5-4_1x04_P5.00mm_Horizontal
- Q1, Q2, Q3, Q4, Q5, Q6: footprint (none) -> Package_TO_SOT_SMD:SC-59; symbol Simulation_SPICE:NMOS -> Transistor_FET:Q_NMOS_GSD
- R1, R10, R11, R12, R13, R14, R15, R2, R3, R4, R5, R6, R7, R8, R9: footprint (none) -> Resistor_SMD:R_0603_1608Metric
- U2: footprint (none) -> Package_TO_SOT_SMD:TO-252-2
Connections:
- net +3.3V: now also MK1.4 (SELECT), C3.1
- net Blue Power: now also Q3.3 (D); no longer Q3.1 (D)
- net GND: now also Q1.2 (S), Q2.2 (S), Q3.2 (S), Q4.2 (S), Q5.2 (S), Q6.2 (S), C3.2; no longer Q1.3 (S), Q2.3 (S), Q3.3 (S), Q4.3 (S), Q5.3 (S), Q6.3 (S)
- net Green Power: now also Q2.3 (D); no longer Q2.1 (D)
- net Red Power: now also Q1.3 (D); no longer Q1.1 (D)
- net at R1.1: now also Q4.3 (D); no longer Q4.1 (D)
- net at R12.2, R15.2: now also Q6.1 (G); no longer Q6.2 (G)
- net at R6.2, R7.2: now also Q2.1 (G); no longer Q2.2 (G)
- net at R11.2, R14.2: now also Q5.1 (G); no longer Q5.2 (G)
- net at R10.2, R13.2: now also Q4.1 (G); no longer Q4.2 (G)
- net at R3.1: now also Q6.3 (D); no longer Q6.1 (D)
- net at R4.2, R5.2: now also Q1.1 (G); no longer Q1.2 (G)
- net at R8.2, R9.2: now also Q3.1 (G); no longer Q3.2 (G)
- net at R2.1: now also Q5.3 (D); no longer Q5.1 (D)
- no-connect marks 20 -> 19

Commit message: Stupid dumb fix
Also did geographical reannotation
Parts:
- renumbered C3 to C1, C1 to C3, Q6 to Q1, Q5 to Q2, Q4 to Q3, Q2 to Q4, Q3 to Q5, Q1 to Q6, R10 to R1, R6 to R10, R9 to R11, R7 to R12, R8 to R13, R5 to R14, R4 to R15, R15 to R2, R1 to R3, R3 to R4, R13 to R5, R14 to R6, R2 to R7, R12 to R8, R11 to R9
Changed lines of the file:
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@@
 		(on_board yes)
 		(dnp no)
-		(property "Reference" "R1"
+		(property "Reference" "R3"
 			(at 132.334 135.636 90)
 			(effects
@@
 			(project ""
 				(path "/3676c628-00eb-4f01-8b84-a1888172e57e"
-					(reference "R1")
+					(reference "R3")
 					(unit 1)
 				)
@@
 		(on_board yes)
 		(dnp no)
-		(property "Reference" "R15"
+		(property "Reference" "R2"
 			(at 95.758 171.45 0)
 			(effects
@@
 			(project "PCB"
 				(path "/3676c628-00eb-4f01-8b84-a1888172e57e"
-					(reference "R15")
+					(reference "R2")
 					(unit 1)
 				)
@@
 		(on_board yes)
 		(dnp no)
-		(property "Reference" "R7"
+		(property "Reference" "R12"
 			(at 46.228 137.16 0)
 			(effects
@@
 			(project "PCB"
 				(path "/3676c628-00eb-4f01-8b84-a1888172e57e"
-					(reference "R7")
+					(reference "R12")
 					(unit 1)
 				)
@@
 		(on_board yes)
 		(dnp no)
-		(property "Reference" "R11"
+		(property "Reference" "R9"
 			(at 86.36 144.272 90)
 			(effects
@@
 			(project "PCB"
 				(path "/3676c628-00eb-4f01-8b84-a1888172e57e"
-					(reference "R11")
+					(reference "R9")
 					(unit 1)
 				)
@@
 		(on_board yes)
 		(dnp no)
-		(property "Reference" "R13"
+		(property "Reference" "R5"
 			(at 95.758 104.14 0)
 			(effects
@@
 			(project "PCB"
 				(path "/3676c628-00eb-4f01-8b84-a1888172e57e"
-					(reference "R13")
+					(reference "R5")
 					(unit 1)
 				)
@@
 		(on_board yes)
 		(dnp no)
-		(property "Reference" "R14"
+		(property "Reference" "R6"
 			(at 95.758 137.16 0)
 			(effects
@@
 			(project "PCB"
 				(path "/3676c628-00eb-4f01-8b84-a1888172e57e"
-					(reference "R14")
+					(reference "R6")
 					(unit 1)
 				)
@@
 		(on_board yes)
 		(dnp no)
-		(property "Reference" "R3"
+		(property "Reference" "R4"
 			(at 132.08 146.558 90)
 			(effects
@@
 			(project ""
 				(path "/3676c628-00eb-4f01-8b84-a1888172e57e"
-					(reference "R3")
+					(reference "R4")
 					(unit 1)
 				)
@@
 		(dnp no)
 		(fields_autoplaced yes)
-		(property "Reference" "Q1"
+		(property "Reference" "Q6"
 			(at 54.61 113.0299 0)
 			(effects
@@
 			(project ""
 				(path "/3676c628-00eb-4f01-8b84-a1888172e57e"
-					(reference "Q1")
+					(reference "Q6")
 					(unit 1)
 				)
@@
 		(on_board yes)
 		(dnp no)
-		(property "Reference" "R4"
+		(property "Reference" "R15"
 			(at 36.83 111.252 90)
 			(effects
@@
 			(project ""
 				(path "/3676c628-00eb-4f01-8b84-a1888172e57e"
-					(reference "R4")
+					(reference "R15")
 					(unit 1)
 				)
@@
 		(on_board yes)
 		(dnp no)
-		(property "Reference" "R10"
+		(property "Reference" "R1"
 			(at 86.36 111.252 90)
 			(effects
@@
 			(project "PCB"
 				(path "/3676c628-00eb-4f01-8b84-a1888172e57e"
-					(reference "R10")
+					(reference "R1")
 					(unit 1)
 				)
@@
 		(dnp no)
 		(fields_autoplaced yes)
-		(property "Reference" "Q6"
+		(property "Reference" "Q1"
 			(at 104.14 180.3399 0)
 			(effects
@@
 			(project "PCB"
 				(path "/3676c628-00eb-4f01-8b84-a1888172e57e"
-					(reference "Q6")
+					(reference "Q1")
 					(unit 1)
 				)
@@
 		(on_board yes)
 		(dnp no)
-		(property "Reference" "R5"
+		(property "Reference" "R14"
 			(at 46.228 104.14 0)
 			(effects
@@
 			(project ""
 				(path "/3676c628-00eb-4f01-8b84-a1888172e57e"
-					(reference "R5")
+					(reference "R14")
 					(unit 1)
 				)
@@
 		(dnp no)
 		(fields_autoplaced yes)
-		(property "Reference" "Q4"
+		(property "Reference" "Q3"
 			(at 104.14 113.0299 0)
 			(effects
@@
 			(project "PCB"
 				(path "/3676c628-00eb-4f01-8b84-a1888172e57e"
-					(reference "Q4")
+					(reference "Q3")
 					(unit 1)
 				)
@@
 		(dnp no)
 		(fields_autoplaced yes)
-		(property "Reference" "Q3"
+		(property "Reference" "Q5"
 			(at 54.61 180.3399 0)
 			(effects
@@
 			(project "PCB"
 				(path "/3676c628-00eb-4f01-8b84-a1888172e57e"
-					(reference "Q3")
+					(reference "Q5")
 					(unit 1)
 				)
@@
 		(dnp no)
 		(fields_autoplaced yes)
-		(property "Reference" "Q2"
+		(property "Reference" "Q4"
 			(at 54.61 146.0499 0)
 			(effects
@@
 			(project "PCB"
 				(path "/3676c628-00eb-4f01-8b84-a1888172e57e"
-					(reference "Q2")
+					(reference "Q4")
 					(unit 1)
 				)
@@
 		(on_board yes)
 		(dnp no)
-		(property "Reference" "R6"
+		(property "Reference" "R10"
 			(at 36.83 144.272 90)
 			(effects
@@
 			(project "PCB"
 				(path "/3676c628-00eb-4f01-8b84-a1888172e57e"
-					(reference "R6")
+					(reference "R10")
 					(unit 1)
 				)
@@
 		(on_board yes)
 		(dnp no)
-		(property "Reference" "C1"
+		(property "Reference" "C3"
 			(at 184.15 46.99 90)
 			(effects
@@
 			(project ""
 				(path "/3676c628-00eb-4f01-8b84-a1888172e57e"
-					(reference "C1")
+					(reference "C3")
 					(unit 1)
 				)
@@
 		(on_board yes)
 		(dnp no)
-		(property "Reference" "R9"
+		(property "Reference" "R11"
 			(at 46.228 171.45 0)
 			(effects
@@
 			(project "PCB"
 				(path "/3676c628-00eb-4f01-8b84-a1888172e57e"
-					(reference "R9")
+					(reference "R11")
 					(unit 1)
 				)
@@
 		(on_board yes)
 		(dnp no)
-		(property "Reference" "R8"
+		(property "Reference" "R13"
 			(at 36.83 178.562 90)
 			(effects
@@
 			(project "PCB"
 				(path "/3676c628-00eb-4f01-8b84-a1888172e57e"
-					(reference "R8")
+					(reference "R13")
 					(unit 1)
 				)
@@
 		(on_board yes)
 		(dnp no)
-		(property "Reference" "R12"
+		(property "Reference" "R8"
 			(at 86.36 178.562 90)
 			(effects
@@
 			(project "PCB"
 				(path "/3676c628-00eb-4f01-8b84-a1888172e57e"
-					(reference "R12")
+					(reference "R8")
 					(unit 1)
 				)
@@
 		(dnp no)
 		(fields_autoplaced yes)
-		(property "Reference" "Q5"
+		(property "Reference" "Q2"
 			(at 104.14 146.0499 0)
 			(effects
@@
 			(project "PCB"
 				(path "/3676c628-00eb-4f01-8b84-a1888172e57e"
-					(reference "Q5")
+					(reference "Q2")
 					(unit 1)
 				)
@@
 		(dnp no)
 		(fields_autoplaced yes)
-		(property "Reference" "C3"
+		(property "Reference" "C1"
 			(at 148.59 85.0899 0)
 			(effects
@@
 			(project ""
 				(path "/3676c628-00eb-4f01-8b84-a1888172e57e"
-					(reference "C3")
+					(reference "C1")
 					(unit 1)
 				)
@@
 		(on_board yes)
 		(dnp no)
-		(property "Reference" "R2"
+		(property "Reference" "R7"
 			(at 132.08 141.224 90)
 			(effects
@@
 			(project ""
 				(path "/3676c628-00eb-4f01-8b84-a1888172e57e"
-					(reference "R2")
+					(reference "R7")
 					(unit 1)
 				)

Commit message: discussed changes
Parts:
- added R7: 84.5, Resistor_SMD:R_0603_1608Metric, symbol Device:R
- renumbered Q5 to Q4, Q4 to Q5, R8 to R1, R7 to R10, R13 to R11, R10 to R12, R15 to R13, R11 to R14, R12 to R15, R14 to R16, R6 to R3, R1 to R4, R9 to R5, R5 to R6, R3 to R8, R4 to R9
Connections:
- net +3.3V: no longer MK1.4 (SELECT)
- net GND: now also MK1.4 (SELECT)
- net PDM Data: now also R7.2; no longer MK1.1 (DATA)
- new net: MK1.1 (DATA), R7.1
Other:
- moved on the sheet: C1, MK1

Commit message: BOM Update
Parts:
- Q1, Q2, Q3: value NMOS -> PJA3432
- Q4, Q5, Q6: value NMOS -> DMN1019
Changed lines of the file:
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@@
 			)
 		)
-		(property "Value" "NMOS"
+		(property "Value" "DMN1019"
 			(at 54.61 115.5699 0)
 			(effects
@@
 			)
 		)
-		(property "Value" "NMOS"
+		(property "Value" "PJA3432"
 			(at 104.14 182.8799 0)
 			(effects
@@
 			)
 		)
-		(property "Value" "NMOS"
+		(property "Value" "PJA3432"
 			(at 104.14 115.5699 0)
 			(effects
@@
 			)
 		)
-		(property "Value" "NMOS"
+		(property "Value" "DMN1019"
 			(at 54.61 182.8799 0)
 			(effects
@@
 			)
 		)
-		(property "Value" "NMOS"
+		(property "Value" "DMN1019"
 			(at 54.61 148.5899 0)
 			(effects
@@
 			)
 		)
-		(property "Value" "NMOS"
+		(property "Value" "PJA3432"
 			(at 104.14 148.5899 0)
 			(effects
